Commit message: change according to my AR3 measurement

File: AR4/description/urdf/ar4_no_gripper.urdf (robot description, URDF)
Before this commit: robot mk3, 9 links, 8 joints
Joints:
- joint joint_3: origin xyz=0 -0.305 0.007 rpy=0 0 3.1416 -> xyz=0 -0.305 0.000 rpy=0 0 3.1416
- joint joint_6: origin xyz=0.000 0 0.041 rpy=0 0 3.1416 -> xyz=0.000 0 0.038 rpy=0 0 3.1416
